File: prototypes/2x2-prototype/hardware/2x2Poc.kicad_sch (KiCad schematic)
At the start: 18 parts, among them SW1 SW_Reed, SW2 SW_Reed, SW3 SW_Reed, SW4 SW_Reed

Commit message: Modified schematics
Parts:
- added R10, R11, R12, R13, R5, R6, R7, R8, R9: 10kΩ, symbol Device:R
Connections:
- net at D52.2 (A): now also D73.2 (A), R10.1, R13.2; no longer A1.22 (D7)
- net at D61.2 (A): now also R6.1; no longer A1.18 (D3)
- net at D71.2 (A): now also R5.1; no longer A1.17 (D2)
- net at A1.19 (D4): now also R7.2; no longer D50.2 (A)
- net at A1.20 (D5): now also R8.2; no longer D72.2 (A)
- net at D62.2 (A): now also R9.1; no longer A1.21 (D6)
- net at A1.23 (D8): now also R13.1; no longer D73.2 (A)
- net at A1.24 (D9): now also R12.1; no longer D63.2 (A)
- net at A1.25 (D10): now also R11.1; no longer D53.2 (A)
- new net: A1.21 (D6), R9.2
- new net: A1.17 (D2), R5.2
- new net: A1.18 (D3), R6.2
- new net: A1.22 (D7), R10.2
- new net: D72.2 (A), R8.1
- new net: D63.2 (A), R12.2
- new net: D50.2 (A), R7.1
- new net: D53.2 (A), R11.2
