File: prototypes/8x8-maquette/hardware/8x8.kicad_sch (KiCad schematic)
At the start: 101 parts, among them J1 Raspberry_Pi_5, SW1 SW_Reed, SW2 SW_Reed, SW3 SW_Reed, SW4 SW_Reed, SW5 SW_Reed, SW6 SW_Reed, SW7 SW_Reed, SW8 SW_Reed, U1 MCP23017_SO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

Commit message: Modified schematics
Parts:
- added R10, R11, R12, R13, R14, R15, R16, R17, R9: 10kΩ, symbol Device:R
Connections:
- net at D16.1 (K), D24.1 (K), D33.1 (K)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: now also R17.1; no longer U2.1 (CA9)
- net at D1.1 (K), D11.2 (A), D12.2 (A)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: now also R16.1; no longer U2.28 (CA8)
- net at D71.1 (K), D72.1 (K), D73.1 (K)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: now also R9.1; no longer U2.21 (CA1)
- net at D61.1 (K), D62.1 (K), D63.1 (K)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: now also R10.1; no longer U2.22 (CA2)
- net at D50.1 (K), D52.1 (K), D53.1 (K)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: now also R11.1; no longer U2.23 (CA3)
- net at D40.1 (K), D41.1 (K), D43.1 (K)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: now also R12.1; no longer U2.24 (CA4)
- net at D30.1 (K), D31.1 (K), D32.1 (K)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: now also R13.1; no longer U2.25 (CA5)
- net at D20.1 (K), D21.1 (K), D22.1 (K)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: now also R14.1; no longer U2.26 (CA6)
- net at D10.1 (K), D11.1 (K), D12.1 (K)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: now also R15.1; no longer U2.27 (CA7)
- new net: R17.2, U2.1 (CA9)
- new net: R9.2, U2.21 (CA1)
- new net: R10.2, U2.22 (CA2)
- new net: R11.2, U2.23 (CA3)
- new net: R12.2, U2.24 (CA4)
- new net: R13.2, U2.25 (CA5)
- new net: R14.2, U2.26 (CA6)
- new net: R15.2, U2.27 (CA7)
- new net: R16.2, U2.28 (CA8)
